File: Arduino-Pro-MiniKiCad.kicad_pcb (KiCad board)
At the start: 2 copper layers, 17.8 x 33 mm, 6 parts, among them U1 ATMEGA328

Commit message: - correction et optimisation
Routing:
- removed copper zone on B.Cu, net (none)
- removed copper zone on F.Cu, net (none)
Changed lines of the file:
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@@
     (uvia_drill 0.1)
   )
-  (module 1X12 (layer B.Cu)
+    (module 1X12 (layer B.Cu)
     (at 156.21 92.3417 270)
     (fp_text reference JP6 (at 3.1623 3.175 360) (layer Eco1.User)
@@
     (pad 2 thru_hole oval (at 2.54 0 180) (size 1.8796 1.8796) (drill 1.016) (layers *.Cu *.Mask))
   )
-  (module TQFP32-08 (layer F.Cu)
+    (module TQFP32-08 (layer F.Cu)
     (at 148.59 107.5817 315)
     (descr "<B>Thin Plasic Quad Flat Package</B> Grid 0.8 mm")
@@
     (pad 32 smd rect (at -2.79908 -4.2926 315) (size 0.5588 1.27) (layers F.Cu F.Paste F.Mask))
   )
-  (module 1X06 (layer B.Cu)
+    (module 1X06 (layer B.Cu)
     (at 142.24 89.789)
     (fp_text reference JP1 (at 5.842 3.937) (layer Eco1.User)
@@
   )
   (gr_line (start 139.7 88.5317) (end 139.7 121.5517) (angle 90) (layer Edge.Cuts) (width 0.2032))
-  (gr_line (start 139.7 121.5517) (end 157.48 121.5517) (angle 90) (layer Edge.Cuts) (width 0.2032))
+    (gr_line (start 139.7 121.5517) (end 157.48 121.5517) (angle 90) (layer Edge.Cuts) (width 0.2032))
   (gr_line (start 157.48 121.5517) (end 157.48 88.5317) (angle 90) (layer Edge.Cuts) (width 0.2032))
   (gr_line (start 157.48 88.5317) (end 139.7 88.5317) (angle 90) (layer Edge.Cuts) (width 0.2032))
-  (gr_circle (center 140.97 112.6617) (end 141.986 112.6617) (layer F.SilkS) (width 0.254))
-  (gr_circle (center 140.97 110.1217) (end 141.986 110.1217) (layer F.SilkS) (width 0.254))
-  (gr_circle (center 140.97 105.0417) (end 141.986 105.0417) (layer F.SilkS) (width 0.254))
-  (gr_circle (center 140.97 120.2817) (end 141.986 120.2817) (layer F.SilkS) (width 0.254))
-  (gr_circle (center 156.21 120.2817) (end 157.226 120.2817) (layer F.SilkS) (width 0.254))
-  (gr_circle (center 156.21 117.7417) (end 157.226 117.7417) (layer F.SilkS) (width 0.254))
-  (zone (net 0) (net_name "") (layer F.Cu) (hatch edge 0.508)
-    (connect_pads (clearance 0.3048))
-    (min_thickness 0.254)
-    (fill (arc_segments 16) (thermal_gap 0.508) (thermal_bridge_width 0.508))
-    (polygon
-      (pts
-        (xy 139.7 88.5317) (xy 157.48 88.5317) (xy 157.48 121.5517) (xy 139.7 121.5517)
-      )
-    )
-  )
-  (zone (net 0) (net_name "") (layer B.Cu) (hatch edge 0.508)
-    (connect_pads (clearance 0.3048))
-    (min_thickness 0.254)
-    (fill (arc_segments 16) (thermal_gap 0.508) (thermal_bridge_width 0.508))
-    (polygon
-      (pts
-        (xy 139.7 88.5317) (xy 157.48 88.5317) (xy 157.48 121.5517) (xy 139.7 121.5517)
-      )
-    )
-  )
 )
